Commit message: updates for actual robot

File: description/ros2_control.xacro (robot description, xacro)
@@ -1,20 +1,35 @@
 <?xml version="1.0"?>
 <robot xmlns:xacro="http://www.ros.org/wiki/xacro">
-    <!--github link-->
-    <!--ros2_control name="GazeboSimSystem" type="system"-->
-    <!--ArtuclatedRobotics-->
-    <!--ros2_control name="GazeboSystem" type="system"-->
-    <!--ChatGipitty-->
-    <!--ros2_control name="GazeboSystem" type="system"-->
-    <ros2_control name="GazeboSystem" type="system">
+    <ros2_control name="RealRobot" type="system">
         <hardware>
-            <!--https://github.com/ros-controls/gz_ros2_control/blob/rolling/gz_ros2_control_demos/urdf/test_diff_drive.xacro.urdf#L149-L179-->
-            <!--plugin>gz_ros2_control/GazeboSimSystem</plugin-->
-            <!--ArtuclatedRobotics-->
-            <!--plugin>gz_ros2_control/DefaultSystem</plugin-->
-            <!--ChatGipitty-->
-            <!--plugin>ros_gz_sim/DefaultSystem</plugin-->
-            <!--CHatchippity-->
-            <!--plugin name="ign_ros2_control::IgnitionROS2ControlPlugin" filename="libign_ros2_control-system.so"/-->
+            <plugin>diffdrive_arduino/DiffDriveArduino</plugin>
+            <param name="left_wheel_name">left_wheel_joint</param>
+            <param name="right_wheel_name">right_wheel_joint</param>
+            <param name="loop_rate">30</param>
+            <param name="device">/dev/serial/by-id/usb-1a86_USB_Serial-if00-port0</param>
+            <param name="baud_rate">57600</param>
+            <param name="timeout">1000</param>
+            <param name="enc_counts_per_rev">3436</param>
+        </hardware>
+        <!-- Note everything below here is the same as the Gazebo one -->
+        <joint name="left_wheel_joint">
+            <command_interface name="velocity">
+                <param name="min">-10</param>
+                <param name="max">10</param>
+            </command_interface>
+            <state_interface name="velocity"/>
+            <state_interface name="position"/>
+        </joint>
+        <joint name="right_wheel_joint">
+            <command_interface name="velocity">
+                <param name="min">-10</param>
+                <param name="max">10</param>
+            </command_interface>
+            <state_interface name="velocity"/>
+            <state_interface name="position"/>
+        </joint>
+    </ros2_control>
+    <!--ros2_control name="GazeboSystem" type="system">
+        <hardware>
             <plugin>gz_ros2_control/GazeboSimSystem</plugin>
         </hardware>
@@ -35,15 +50,6 @@
             <state_interface name="position"/>
         </joint>
-    </ros2_control>
+    </ros2_control-->
     <gazebo>
-        <!--https://github.com/ros-controls/gz_ros2_control/blob/rolling/gz_ros2_control_demos/urdf/test_diff_drive.xacro.urdf#L149-L179-->
-        <!--plugin filename="gz_ros2_control-system" name="gz_ros2_control::GazeboSimROS2ControlPlugin"-->
-        <!--ArtuclatedRobotics-->
-        <!--plugin name="gz_ros2_control::GazeboSimROS2ControlPlugin" filename="libgz_ros2_control-system.so"-->
-        <!--ChatGipitty-->
-        <!--plugin name="ros_gz_sim::DefaultSystem" filename="libros_gz_sim_ros2_control-system.so"-->
-        <!--ChatGipitty but launches without error-->
-        <!--plugin name="ign_ros2_control::IgnitionROS2ControlPlugin" filename="libros_gz_sim_ros2_control-system.so"-->
-        <!--plugin name="ros2_control" filename="libign_ros2_control-system.so"-->
         <plugin name="gz_ros2_control::GazeboSimROS2ControlPlugin" filename="libgz_ros2_control-system.so">
             <parameters>$(find my_bot)/config/my_controllers.yaml</parameters>
