Commit message: rotate lidar, add lidar to robot launch

File: description/lidar.xacro (robot description, xacro)
@@ -4,5 +4,5 @@
         <parent link="chassis"/>
         <child link="laser_frame"/>
-        <origin xyz="0.122 0 0.175" rpy="0 0 0"/>
+        <origin xyz="0.122 0 0.175" rpy="0 0 ${pi}"/>
     </joint>
     <link name="laser_frame">
@@ -14,5 +14,5 @@
         </visual>
         <visual>
-            <origin xyz="0 0 -0.05"/>
+            <origin xyz="0 0 -0.05" rpy="0 0 ${pi/4}"/>
             <geometry>
                 <cylinder radius="0.01" length="0.1"/>
@@ -26,5 +26,5 @@
         </collision>
         <xacro:inertial_cylinder mass="0.1" length="0.04" radius="0.05">
-            <origin xyz="0 0 0" rpy="0 0 0"/>
+            <origin xyz="0 0 0" rpy="0 0 ${pi/4}"/>
         </xacro:inertial_cylinder>
     </link>
