Commit message: troubleshooting why gazebo wont launch with ros2 control

File: description/robot_core.xacro (robot description, xacro)
@@ -120,4 +120,7 @@
             <material name="black"/>
         </collision>
+        <xacro:inertial_sphere mass="0.1" radius="0.05">
+            <origin xyz="0 0 0" rpy="0 0 0"/>
+        </xacro:inertial_sphere>
     </link>
     <gazebo reference="caster_wheel">

File: description/ros2_control.xacro (robot description, xacro)
@@ -1,7 +1,21 @@
 <?xml version="1.0"?>
 <robot xmlns:xacro="http://www.ros.org/wiki/xacro">
+    <!--github link-->
+    <!--ros2_control name="GazeboSimSystem" type="system"-->
+    <!--ArtuclatedRobotics-->
+    <!--ros2_control name="GazeboSystem" type="system"-->
+    <!--ChatGipitty-->
+    <!--ros2_control name="GazeboSystem" type="system"-->
     <ros2_control name="GazeboSystem" type="system">
         <hardware>
-            <plugin>ros_gz_sim/DefaultSystem</plugin>
+            <!--https://github.com/ros-controls/gz_ros2_control/blob/rolling/gz_ros2_control_demos/urdf/test_diff_drive.xacro.urdf#L149-L179-->
+            <!--plugin>gz_ros2_control/GazeboSimSystem</plugin-->
+            <!--ArtuclatedRobotics-->
+            <!--plugin>gz_ros2_control/DefaultSystem</plugin-->
+            <!--ChatGipitty-->
+            <!--plugin>ros_gz_sim/DefaultSystem</plugin-->
+            <!--CHatchippity-->
+            <!--plugin name="ign_ros2_control::IgnitionROS2ControlPlugin" filename="libign_ros2_control-system.so"/-->
+            <plugin>gz_ros2_control/GazeboSimSystem</plugin>
         </hardware>
         <joint name="left_wheel_joint">
@@ -23,5 +37,14 @@
     </ros2_control>
     <gazebo>
-        <plugin name="ros_gz_sim::DefaultSystem" filename="libros_gz_sim_ros2_control-system.so">
+        <!--https://github.com/ros-controls/gz_ros2_control/blob/rolling/gz_ros2_control_demos/urdf/test_diff_drive.xacro.urdf#L149-L179-->
+        <!--plugin filename="gz_ros2_control-system" name="gz_ros2_control::GazeboSimROS2ControlPlugin"-->
+        <!--ArtuclatedRobotics-->
+        <!--plugin name="gz_ros2_control::GazeboSimROS2ControlPlugin" filename="libgz_ros2_control-system.so"-->
+        <!--ChatGipitty-->
+        <!--plugin name="ros_gz_sim::DefaultSystem" filename="libros_gz_sim_ros2_control-system.so"-->
+        <!--ChatGipitty but launches without error-->
+        <!--plugin name="ign_ros2_control::IgnitionROS2ControlPlugin" filename="libros_gz_sim_ros2_control-system.so"-->
+        <!--plugin name="ros2_control" filename="libign_ros2_control-system.so"-->
+        <plugin name="gz_ros2_control::GazeboSimROS2ControlPlugin" filename="libgz_ros2_control-system.so">
             <parameters>$(find my_bot)/config/my_controllers.yaml</parameters>
             <parameters>$(find my_bot)/config/gaz_ros2_ctl_use_sim.yaml</parameters>

Commit message: robot core tweaks

File: description/robot_core.xacro (robot description, xacro)
@@ -51,5 +51,5 @@
     <parent link="base_link"/>
     <child link="left_wheel"/>
-    <origin xyz="0 0.175 0" rpy="-${pi/2} 0 0"/>
+    <origin xyz="0.1 0.175 0" rpy="-${pi/2} 0 0"/>
     <axis xyz="0 0 1"/>
     </joint>
@@ -67,7 +67,7 @@
             <material name="blue"/>
         </collision>
-        <xacro:inertial_cylinder mass="0.1" length="0.05" radius="0.05">
+        <xacro:inertial_sphere mass="0.1" radius="0.05">
             <origin xyz="0 0 0" rpy="0 0 0"/>
-        </xacro:inertial_cylinder>
+        </xacro:inertial_sphere>
     </link>
     <gazebo reference="left_wheel">
@@ -78,5 +78,5 @@
         <parent link="base_link"/>
         <child link="right_wheel"/>
-        <origin xyz="0 -0.175 0" rpy="${pi/2} 0 0"/>
+        <origin xyz="0.1 -0.175 0" rpy="${pi/2} 0 0"/>
         <axis xyz="0 0 -1"/>
     </joint>

Commit message: added base link

File: description/robot_core.xacro (robot description, xacro)
@@ -20,4 +20,10 @@
     <link name="base_link">
     </link>
+    <!-- BASE_FOOTPRINT LINK-->
+    <joint name="base_footprint_joint" type="fixed">
+        <parent link="base_link"/>
+        <child link="base_footprint"/>
+        <origin xyz="0 0 0" rpy="0 0 0">
+    </joint>
     <!-- CHASSIS -->
     <joint name="chassis_joint" type="fixed">

Commit message: robot core fix

File: description/robot_core.xacro (robot description, xacro)
@@ -21,9 +21,11 @@
     </link>
     <!-- BASE_FOOTPRINT LINK-->
-    <!--joint name="base_footprint_joint" type="fixed">
+    <joint name="base_footprint_joint" type="fixed">
         <parent link="base_link"/>
         <child link="base_footprint"/>
         <origin xyz="0 0 0" rpy="0 0 0"/>
-    </joint-->
+    </joint>
+    <link name="base_footprint">
+    </link>
     <!-- CHASSIS -->
     <joint name="chassis_joint" type="fixed">

Commit message: updates

File: description/robot_core.xacro (robot description, xacro)
@@ -65,5 +65,5 @@
         <visual>
             <geometry>
-                <cylinder length="0.04" radius="0.05" />
+                <cylinder length="0.04" radius="0.045" />
             </geometry>
             <material name="blue"/>
@@ -71,9 +71,9 @@
         <collision>
             <geometry>
-                <cylinder length="0.04" radius="0.05" />
+                <cylinder length="0.04" radius="0.045" />
             </geometry>
             <material name="blue"/>
         </collision>
-        <xacro:inertial_sphere mass="0.1" radius="0.05">
+        <xacro:inertial_sphere mass="0.1" radius="0.045">
             <origin xyz="0 0 0" rpy="0 0 0"/>
         </xacro:inertial_sphere>
@@ -92,5 +92,5 @@
         <visual>
             <geometry>
-                <cylinder length="0.04" radius="0.05" />
+                <cylinder length="0.04" radius="0.045" />
             </geometry>
             <material name="blue"/>
@@ -98,9 +98,9 @@
             <collision>
             <geometry>
-                <cylinder length="0.04" radius="0.05" />
+                <cylinder length="0.04" radius="0.045" />
             </geometry>
             <material name="blue"/>
         </collision>
-        <xacro:inertial_sphere mass="0.1" radius="0.05">
+        <xacro:inertial_sphere mass="0.1" radius="0.045">
             <origin xyz="0 0 0" rpy="0 0 0"/>
         </xacro:inertial_sphere>

File: description/ros2_control.xacro (robot description, xacro)
@@ -11,5 +11,5 @@
                 <param name="baud_rate">57600</param>
                 <param name="timeout_ms">1000</param>
-                <param name="enc_counts_per_rev">3436</param>
+                <param name="enc_counts_per_rev">1950</param>
             </hardware>
             <joint name="left_wheel_joint">

Commit message: updates to dimensions

File: description/robot_core.xacro (robot description, xacro)
@@ -65,5 +65,5 @@
         <visual>
             <geometry>
-                <cylinder length="0.04" radius="0.045" />
+                <cylinder length="0.04" radius="0.035" />
             </geometry>
             <material name="blue"/>
@@ -71,9 +71,9 @@
         <collision>
             <geometry>
-                <cylinder length="0.04" radius="0.045" />
+                <cylinder length="0.04" radius="0.035" />
             </geometry>
             <material name="blue"/>
         </collision>
-        <xacro:inertial_sphere mass="0.1" radius="0.045">
+        <xacro:inertial_sphere mass="0.1" radius="0.035">
             <origin xyz="0 0 0" rpy="0 0 0"/>
         </xacro:inertial_sphere>
@@ -92,5 +92,5 @@
         <visual>
             <geometry>
-                <cylinder length="0.04" radius="0.045" />
+                <cylinder length="0.04" radius="0.035" />
             </geometry>
             <material name="blue"/>
@@ -98,9 +98,9 @@
             <collision>
             <geometry>
-                <cylinder length="0.04" radius="0.045" />
+                <cylinder length="0.04" radius="0.035" />
             </geometry>
             <material name="blue"/>
         </collision>
-        <xacro:inertial_sphere mass="0.1" radius="0.045">
+        <xacro:inertial_sphere mass="0.1" radius="0.035">
             <origin xyz="0 0 0" rpy="0 0 0"/>
         </xacro:inertial_sphere>
